Commit message: Add initial link4 vertical compensation ROS2 node

File: src/ur10e_cylinder/urdf/ur10e_cylinder.urdf (robot description, URDF)
Before this commit: robot ur10e_cylinder, 7 links, 6 joints
Joints:
- joint elbow_joint: limit lower=-3.14 upper=3.14 effort=100 velocity=1.0 -> lower=0 upper=2.5 effort=100 velocity=1.0
- joint shoulder_lift_joint: limit lower=-3.14 upper=3.14 effort=100 velocity=1.0 -> lower=0 upper=2.5 effort=100 velocity=1.0; origin xyz=0 0 0.15 rpy=0 1.5708 0 -> xyz=0 0 0.15 rpy=0 0 0
- joint shoulder_pan_joint: limit lower=-6.28 upper=6.28 effort=100 velocity=1.0 -> lower=-3.14 upper=3.14 effort=100 velocity=1.0
- joint wrist_1_joint: limit lower=-6.28 upper=6.28 effort=50 velocity=1.0 -> lower=-3.14 upper=3.14 effort=50 velocity=1.0; origin xyz=0 0 0.572 rpy=0 1.5708 0 -> xyz=0 0 0.572 rpy=0 0 0
- joint wrist_2_joint: limit lower=-6.28 upper=6.28 effort=50 velocity=1.0 -> lower=-1.57 upper=1.57 effort=50 velocity=1.0; origin xyz=0 0 0.163 rpy=0 -1.5708 0 -> xyz=0 0 0.163 rpy=0 0 0
- joint wrist_3_joint: limit lower=-6.28 upper=6.28 effort=50 velocity=1.0 -> lower=-3.14 upper=3.14 effort=50 velocity=1.0

File: src/ur10e_moveit_config/config/ur10e_cylinder.ros2_control.xacro (robot description, xacro)
@@ -7,6 +7,4 @@
                 <!-- By default, set up controllers for simulation. This won't work on real hardware -->
                 <plugin>mock_components/GenericSystem</plugin>
-                <param name="fake_sensor_commands">false</param>
-                <param name="state_following_offset">0.0</param>
             </hardware>
             <joint name="shoulder_pan_joint">

Commit message: Working MoveIt joint-point sequence before MoveItPy migration

File: src/ur10e_cylinder/urdf/ur10e_cylinder.urdf (robot description, URDF)
Before this commit: robot ur10e_cylinder, 7 links, 6 joints
Links:
- added link obstacle_cylinder; collision cylinder length=0.7 radius=0.3; visual cylinder length=0.7 radius=0.3
- added link world
Joints:
- added joint world_to_base: type fixed, parent world, child base_link, origin xyz=0 0 0 rpy=0 0 4.71239
- added joint world_to_obstacle: type fixed, parent world, child obstacle_cylinder, origin xyz=0.45 -0.3 0.35 rpy=0 0 0
- joint elbow_joint: limit lower=0 upper=2.5 effort=100 velocity=1.0 -> lower=-2.224 upper=2.224 effort=100 velocity=1.0
- joint shoulder_lift_joint: limit lower=0 upper=2.5 effort=100 velocity=1.0 -> lower=-3.14 upper=3.14 effort=100 velocity=1.0; origin xyz=0 0 0.15 rpy=0 0 0 -> xyz=0 0 0.15 rpy=0 1.5708 0
- joint wrist_1_joint: limit lower=-3.14 upper=3.14 effort=50 velocity=1.0 -> lower=-2.224 upper=2.224 effort=50 velocity=1.0

Commit message: Working UR10e cylinder model with corrected wrist and end effector alignment

File: src/ur10e_cylinder/urdf/ur10e_cylinder.urdf (robot description, URDF)
Before this commit: robot ur10e_cylinder, 9 links, 8 joints
Links:
- link tool0: geometry collision box size=0.1 0.02 0.02; visual box size=0.1 0.02 0.02
Joints:
- joint wrist_1_joint: limit lower=-2.224 upper=2.224 effort=50 velocity=1.0 -> lower=-3.14 upper=3.14 effort=50 velocity=1.0
- joint wrist_2_joint: axis 1 0 0 -> 0 0 1; limit lower=-1.57 upper=1.57 effort=50 velocity=1.0 -> lower=-3.14 upper=3.14 effort=50 velocity=1.0
- joint wrist_3_joint: axis 0 0 1 -> 0 1 0; origin xyz=0 0 0.115 rpy=0 0 0 -> xyz=0 0.115 0 rpy=0 0 0

Commit message: trial

File: src/ur10e_cylinder/urdf/ur10e_cylinder.urdf (robot description, URDF)
Before this commit: robot ur10e_cylinder, 9 links, 8 joints
Links:
- removed link obstacle_cylinder
- added link obstacle_1; collision cylinder length=0.2 radius=0.3; visual cylinder length=0.2 radius=0.3
- added link obstacle_2; collision cylinder length=0.2 radius=0.3; visual cylinder length=0.2 radius=0.3
- added link obstacle_3; collision cylinder length=0.2 radius=0.3; visual cylinder length=0.2 radius=0.3
- added link obstacle_4; collision cylinder length=0.2 radius=0.3; visual cylinder length=0.2 radius=0.3
- added link obstacle_5; collision cylinder length=0.2 radius=0.3; visual cylinder length=0.2 radius=0.3
- added link obstacle_6; collision cylinder length=0.2 radius=0.3; visual cylinder length=0.2 radius=0.3
- added link obstacle_7; collision cylinder length=0.2 radius=0.3; visual cylinder length=0.2 radius=0.3
- added link obstacle_8; collision cylinder length=0.2 radius=0.3; visual cylinder length=0.2 radius=0.3
- link link2: geometry collision cylinder length=0.613 radius=0.05; visual cylinder length=0.613 radius=0.05
- link link3: geometry collision cylinder length=0.571 radius=0.045; visual cylinder length=0.571 radius=0.045
- link link4: geometry collision cylinder length=0.74 radius=0.04; visual cylinder length=0.174 radius=0.04
- link link5: geometry collision cylinder length=0.120 radius=0.035; visual cylinder length=0.120 radius=0.035
- link tool0: geometry collision box size=0.1 0.02 0.02; visual box size=0.08 0.02 0.02
Joints:
- removed joint world_to_obstacle
- added joint world_to_obstacle_1: type fixed, parent world, child obstacle_1, origin xyz=0.45 -0.3 0.1 rpy=0 0 0
- added joint world_to_obstacle_2: type fixed, parent world, child obstacle_2, origin xyz=0.45 -0.3 0.3 rpy=0 0 0
- added joint world_to_obstacle_3: type fixed, parent world, child obstacle_3, origin xyz=0.45 -0.3 0.5 rpy=0 0 0
- added joint world_to_obstacle_4: type fixed, parent world, child obstacle_4, origin xyz=0.45 -0.3 0.7 rpy=0 0 0
- added joint world_to_obstacle_5: type fixed, parent world, child obstacle_5, origin xyz=0.45 -0.3 0.9 rpy=0 0 0
- added joint world_to_obstacle_6: type fixed, parent world, child obstacle_6, origin xyz=0.45 -0.3 1.1 rpy=0 0 0
- added joint world_to_obstacle_7: type fixed, parent world, child obstacle_7, origin xyz=0.45 -0.3 1.3 rpy=0 0 0
- added joint world_to_obstacle_8: type fixed, parent world, child obstacle_8, origin xyz=0.45 -0.3 1.5 rpy=0 0 0
- joint elbow_joint: origin xyz=0 0 0.612 rpy=0 0 0 -> xyz=0 0 0.613 rpy=0 0 0
- joint wrist_1_joint: origin xyz=0 0 0.572 rpy=0 0 0 -> xyz=0 0 0.571 rpy=0 0 0
- joint wrist_2_joint: origin xyz=0 0 0.163 rpy=0 0 0 -> xyz=0 0 0.174 rpy=0 0 0
- joint wrist_3_joint: origin xyz=0 0.115 0 rpy=0 0 0 -> xyz=0 0.120 0 rpy=0 0 0

Commit message: trial1

File: src/ur10e_cylinder/urdf/ur10e_cylinder.urdf (robot description, URDF)
Before this commit: robot ur10e_cylinder, 16 links, 15 joints
Joints:
- joint world_to_base: origin xyz=0 0 0 rpy=0 0 4.71239 -> xyz=0 0 0.6 rpy=0 0 4.71239

Commit message: working one with going back to exact position

File: src/ur10e_cylinder/urdf/ur10e_cylinder.urdf (robot description, URDF)
Before this commit: robot ur10e_cylinder, 16 links, 15 joints
Links:
- added link camera_link; collision cylinder length=0.08 radius=0.02; visual cylinder length=0.08 radius=0.02
- link base_link: geometry collision cylinder length=0.18 radius=0.06; visual cylinder length=0.18 radius=0.06
- link link4: geometry collision cylinder length=0.174 radius=0.04; visual cylinder length=0.174 radius=0.04
- link obstacle_1: geometry collision cylinder length=0.2 radius=0.15; visual cylinder length=0.2 radius=0.15
- link obstacle_2: geometry collision cylinder length=0.2 radius=0.15; visual cylinder length=0.2 radius=0.15
- link obstacle_3: geometry collision cylinder length=0.2 radius=0.15; visual cylinder length=0.2 radius=0.15
- link obstacle_4: geometry collision cylinder length=0.2 radius=0.15; visual cylinder length=0.2 radius=0.15
- link obstacle_5: geometry collision cylinder length=0.2 radius=0.15; visual cylinder length=0.2 radius=0.15
- link obstacle_6: geometry collision cylinder length=0.2 radius=0.15; visual cylinder length=0.2 radius=0.15
- link obstacle_7: geometry collision cylinder length=0.2 radius=0.15; visual cylinder length=0.2 radius=0.15
- link obstacle_8: geometry collision cylinder length=0.2 radius=0.15; visual cylinder length=0.2 radius=0.15
Joints:
- added joint wrist_camera_joint: type fixed, parent link4, child camera_link, origin xyz=0 0 0.1
- joint elbow_joint: limit lower=-2.224 upper=2.224 effort=100 velocity=1.0 -> lower=-6.28 upper=6.28 effort=100 velocity=1.0; origin xyz=0 0 0.613 rpy=0 0 0 -> xyz=0 -0.095 0.613
- joint shoulder_lift_joint: limit lower=-3.14 upper=3.14 effort=100 velocity=1.0 -> lower=-6.28 upper=6.28 effort=100 velocity=1.0; origin xyz=0 0 0.15 rpy=0 1.5708 0 -> xyz=0 0.11 0.15 rpy=0 1.5708 0
- joint shoulder_pan_joint: limit lower=-3.14 upper=3.14 effort=100 velocity=1.0 -> lower=0.00 upper=1.57 effort=100 velocity=1.0; origin xyz=0 0 0.127 rpy=0 0 0 -> xyz=0 0 0.127
- joint world_to_obstacle_1: origin xyz=0.45 -0.3 0.1 rpy=0 0 0 -> xyz=0.45 -0.3 0.1
- joint world_to_obstacle_2: origin xyz=0.45 -0.3 0.3 rpy=0 0 0 -> xyz=0.45 -0.3 0.3
- joint world_to_obstacle_3: origin xyz=0.45 -0.3 0.5 rpy=0 0 0 -> xyz=0.45 -0.3 0.5
- joint world_to_obstacle_4: origin xyz=0.45 -0.3 0.7 rpy=0 0 0 -> xyz=0.45 -0.3 0.7
- joint world_to_obstacle_5: origin xyz=0.45 -0.3 0.9 rpy=0 0 0 -> xyz=0.45 -0.3 0.9
- joint world_to_obstacle_6: origin xyz=0.45 -0.3 1.1 rpy=0 0 0 -> xyz=0.45 -0.3 1.1
- joint world_to_obstacle_7: origin xyz=0.45 -0.3 1.3 rpy=0 0 0 -> xyz=0.45 -0.3 1.3
- joint world_to_obstacle_8: origin xyz=0.45 -0.3 1.5 rpy=0 0 0 -> xyz=0.45 -0.3 1.5
- joint wrist_1_joint: limit lower=-3.14 upper=3.14 effort=50 velocity=1.0 -> lower=-6.28 upper=6.28 effort=50 velocity=1.0; origin xyz=0 0 0.571 rpy=0 0 0 -> xyz=0 0.08 0.571
- joint wrist_2_joint: limit lower=-3.14 upper=3.14 effort=50 velocity=1.0 -> lower=-6.28 upper=6.28 effort=50 velocity=1.0; origin xyz=0 0 0.174 rpy=0 0 0 -> xyz=0 0 0.174
- joint wrist_3_joint: limit lower=-3.14 upper=3.14 effort=50 velocity=1.0 -> lower=-6.28 upper=6.28 effort=50 velocity=1.0; origin xyz=0 0.120 0 rpy=0 0 0 -> xyz=0 0.120 0

Commit message: cylinder removed from urdf added to move_to_pose.py

File: src/ur10e_cylinder/urdf/ur10e_cylinder.urdf (robot description, URDF)
Before this commit: robot ur10e_cylinder, 17 links, 16 joints
Links:
- removed link obstacle_1
- removed link obstacle_2
- removed link obstacle_3
- removed link obstacle_4
- removed link obstacle_5
- removed link obstacle_6
- removed link obstacle_7
- removed link obstacle_8
- link tool0: geometry collision box size=0.04 0.02 0.02; visual box size=0.04 0.02 0.02
Joints:
- removed joint world_to_obstacle_1
- removed joint world_to_obstacle_2
- removed joint world_to_obstacle_3
- removed joint world_to_obstacle_4
- removed joint world_to_obstacle_5
- removed joint world_to_obstacle_6
- removed joint world_to_obstacle_7
- removed joint world_to_obstacle_8

Commit message: with gripper urdf

File: src/ur10e_cylinder/urdf/ur10e_cylinder.urdf (robot description, URDF)
Before this commit: robot ur10e_cylinder, 8 links, 7 joints
Links:
- added link gripper_base_link; visual box size=0.06 0.02 0.02
- added link left_finger; visual box size=0.02 0.01 0.06
- added link right_finger; visual box size=0.02 0.01 0.06
Joints:
- added joint left_finger_joint: type prismatic, parent gripper_base_link, child left_finger, origin xyz=0 0.025 0, axis 0 1 0, limit lower=0.0 upper=0.02 effort=10 velocity=0.1
- added joint right_finger_joint: type prismatic, parent gripper_base_link, child right_finger, origin xyz=0 -0.025 0, axis 0 -1 0, limit lower=0.0 upper=0.02 effort=10 velocity=0.1
- added joint tool0_to_gripper: type fixed, parent tool0, child gripper_base_link, origin xyz=0 0 0 rpy=-1.5708 0 0

Commit message: urdf fixed for gripper,before performing moveit assistant

File: src/ur10e_cylinder/urdf/ur10e_cylinder.urdf (robot description, URDF)
Before this commit: robot ur10e_cylinder, 11 links, 10 joints
Links:
- link gripper_base_link: geometry visual box size=0.02 0.06 0.02
- link left_finger: geometry visual box size=0.02 0.01 0.05
- link right_finger: geometry visual box size=0.02 0.01 0.05
Joints:
- joint left_finger_joint: axis 0 1 0 -> 0 -1 0
- joint right_finger_joint: mimic (none) -> joint=left_finger_joint multiplier=-1.0
- joint tool0_to_gripper: origin xyz=0 0 0 rpy=-1.5708 0 0 -> xyz=0 0.03 0 rpy=-1.5708 0 0
