Commit message: with ptp

File: src/ur10e_cylinder/urdf/demo.urdf (robot description, URDF)
Before this commit: robot ur10e_cylinder, 8 links, 7 joints
Links:
- added link camera_link; collision cylinder length=0.08 radius=0.02; visual cylinder length=0.08 radius=0.02
- added link obstacle_1; collision cylinder length=0.2 radius=0.2; visual cylinder length=0.2 radius=0.2
- added link obstacle_2; collision cylinder length=0.2 radius=0.2; visual cylinder length=0.2 radius=0.2
- added link obstacle_3; collision cylinder length=0.2 radius=0.2; visual cylinder length=0.2 radius=0.2
- added link obstacle_4; collision cylinder length=0.2 radius=0.2; visual cylinder length=0.2 radius=0.2
- added link obstacle_5; collision cylinder length=0.2 radius=0.2; visual cylinder length=0.2 radius=0.2
- added link obstacle_6; collision cylinder length=0.2 radius=0.2; visual cylinder length=0.2 radius=0.2
- added link obstacle_7; collision cylinder length=0.2 radius=0.2; visual cylinder length=0.2 radius=0.2
- added link obstacle_8; collision cylinder length=0.2 radius=0.2; visual cylinder length=0.2 radius=0.2
Joints:
- added joint world_to_obstacle_1: type fixed, parent world, child obstacle_1, origin xyz=0.45 -0.3 0.1 rpy=0 0 0
- added joint world_to_obstacle_2: type fixed, parent world, child obstacle_2, origin xyz=0.45 -0.3 0.3 rpy=0 0 0
- added joint world_to_obstacle_3: type fixed, parent world, child obstacle_3, origin xyz=0.45 -0.3 0.5 rpy=0 0 0
- added joint world_to_obstacle_4: type fixed, parent world, child obstacle_4, origin xyz=0.45 -0.3 0.7 rpy=0 0 0
- added joint world_to_obstacle_5: type fixed, parent world, child obstacle_5, origin xyz=0.45 -0.3 0.9 rpy=0 0 0
- added joint world_to_obstacle_6: type fixed, parent world, child obstacle_6, origin xyz=0.45 -0.3 1.1 rpy=0 0 0
- added joint world_to_obstacle_7: type fixed, parent world, child obstacle_7, origin xyz=0.45 -0.3 1.3 rpy=0 0 0
- added joint world_to_obstacle_8: type fixed, parent world, child obstacle_8, origin xyz=0.45 -0.3 1.5 rpy=0 0 0
- added joint wrist_camera_joint: type fixed, parent link4, child camera_link, origin xyz=0 0 0.1

Commit message: working code with twist working tilt not enabled leaves as obstacle

File: src/ur10e_cylinder/urdf/demo.urdf (robot description, URDF)
Before this commit: robot ur10e_cylinder, 36 links, 35 joints
Links:
- link plant_base: geometry collision cylinder length=1.35 radius=0.015; visual cylinder length=1.35 radius=0.015
Joints:
- joint leaf_10_joint: origin xyz=0.5053 -0.3275 0.7625 rpy=0 0 2.00713 -> xyz=0.5053 -0.2725 0.7625 rpy=0 0 2.00713
- joint leaf_11_joint: origin xyz=0.4474 -0.3502 0.8188 rpy=0 0 4.40714 -> xyz=0.4474 -0.2498 0.8188 rpy=0 0 4.40714
- joint leaf_12_joint: origin xyz=0.3951 -0.2918 0.8750 rpy=0 0 0.52360 -> xyz=0.3951 -0.3082 0.8750 rpy=0 0 0.52360
- joint leaf_13_joint: origin xyz=0.4744 -0.2688 0.9313 rpy=0 0 2.92360 -> xyz=0.4744 -0.3312 0.9313 rpy=0 0 2.92343
- joint leaf_14_joint: origin xyz=0.5054 -0.3221 0.9875 rpy=0 0 5.32325 -> xyz=0.5054 -0.2779 0.9875 rpy=0 0 5.32325
- joint leaf_15_joint: origin xyz=0.4510 -0.3490 1.0438 rpy=0 0 1.43990 -> xyz=0.4510 -0.2510 1.0438 rpy=0 0 1.43990
- joint leaf_16_joint: origin xyz=0.3944 -0.2941 1.1000 rpy=0 0 3.83972 -> xyz=0.3944 -0.3059 1.1000 rpy=0 0 3.83972
- joint leaf_17_joint: origin xyz=0.4716 -0.2705 1.1563 rpy=0 0 6.23972 -> xyz=0.4716 -0.3295 1.1563 rpy=0 0 6.23955
- joint leaf_18_joint: origin xyz=0.5052 -0.3168 1.2125 rpy=0 0 2.35619 -> xyz=0.5052 -0.2832 1.2125 rpy=0 0 2.35619
- joint leaf_19_joint: origin xyz=0.4544 -0.3477 1.2688 rpy=0 0 4.75619 -> xyz=0.4544 -0.2523 1.2688 rpy=0 0 4.75602
- joint leaf_1_joint: origin xyz=0.4910 -0.2620 0.2563 rpy=0 0 5.54306 -> xyz=0.4910 -0.3380 0.2563 rpy=0 0 5.54142
- joint leaf_20_joint: origin xyz=0.3937 -0.2963 1.3250 rpy=0 0 0.87266 -> xyz=0.3937 -0.3037 1.3250 rpy=0 0 0.87266
- joint leaf_21_joint: origin xyz=0.4688 -0.2722 1.3813 rpy=0 0 3.27249 -> xyz=0.4688 -0.3278 1.3813 rpy=0 0 3.27249
- joint leaf_22_joint: origin xyz=0.5048 -0.3115 1.4375 rpy=0 0 5.67232 -> xyz=0.5048 -0.2885 1.4375 rpy=0 0 5.67232
- joint leaf_23_joint: origin xyz=0.4577 -0.3464 1.4938 rpy=0 0 1.78897 -> xyz=0.4577 -0.2536 1.4938 rpy=0 0 1.78897
- joint leaf_2_joint: origin xyz=0.5042 -0.3385 0.3125 rpy=0 0 1.65806 -> xyz=0.5042 -0.2615 0.3125 rpy=0 0 1.65806
- joint leaf_3_joint: origin xyz=0.4399 -0.3522 0.3688 rpy=0 0 4.05777 -> xyz=0.4399 -0.2478 0.3688 rpy=0 0 4.05789
- joint leaf_4_joint: origin xyz=0.3967 -0.2874 0.4250 rpy=0 0 0.17453 -> xyz=0.3967 -0.3126 0.4250 rpy=0 0 0.17453
- joint leaf_5_joint: origin xyz=0.4803 -0.2655 0.4813 rpy=0 0 2.57453 -> xyz=0.4803 -0.3345 0.4813 rpy=0 0 2.57436
- joint leaf_6_joint: origin xyz=0.5050 -0.3328 0.5375 rpy=0 0 4.97419 -> xyz=0.5050 -0.2672 0.5375 rpy=0 0 4.97419
- joint leaf_7_joint: origin xyz=0.4438 -0.3513 0.5938 rpy=0 0 1.09083 -> xyz=0.4438 -0.2487 0.5938 rpy=0 0 1.09083
- joint leaf_8_joint: origin xyz=0.3959 -0.2896 0.6500 rpy=0 0 3.49066 -> xyz=0.3959 -0.3104 0.6500 rpy=0 0 3.49066
- joint leaf_9_joint: origin xyz=0.4773 -0.2671 0.7063 rpy=0 0 5.89049 -> xyz=0.4773 -0.3329 0.7063 rpy=0 0 5.89049
- joint shoulder_pan_joint: limit lower=0.00 upper=3.14 effort=100 velocity=1.0 -> lower=0.0 upper=3.14 effort=100 velocity=1.0
