Commit message: https://github.com/himalthilakanp/ur10_ws

File: src/ur10e_moveit_config/config/ur10e_cylinder.ros2_control.xacro (robot description, xacro)
@@ -13,5 +13,4 @@
                   <param name="initial_value">${initial_positions['shoulder_pan_joint']}</param>
                 </state_interface>
-                <state_interface name="velocity"/>
             </joint>
             <joint name="shoulder_lift_joint">
@@ -20,5 +19,4 @@
                   <param name="initial_value">${initial_positions['shoulder_lift_joint']}</param>
                 </state_interface>
-                <state_interface name="velocity"/>
             </joint>
             <joint name="elbow_joint">
@@ -27,5 +25,4 @@
                   <param name="initial_value">${initial_positions['elbow_joint']}</param>
                 </state_interface>
-                <state_interface name="velocity"/>
             </joint>
             <joint name="wrist_1_joint">
@@ -34,5 +31,4 @@
                   <param name="initial_value">${initial_positions['wrist_1_joint']}</param>
                 </state_interface>
-                <state_interface name="velocity"/>
             </joint>
             <joint name="wrist_2_joint">
@@ -41,5 +37,4 @@
                   <param name="initial_value">${initial_positions['wrist_2_joint']}</param>
                 </state_interface>
-                <state_interface name="velocity"/>
             </joint>
             <joint name="wrist_3_joint">
@@ -48,5 +43,10 @@
                   <param name="initial_value">${initial_positions['wrist_3_joint']}</param>
                 </state_interface>
-                <state_interface name="velocity"/>
+            </joint>
+            <joint name="left_finger_joint">
+                <command_interface name="position"/>
+                <state_interface name="position">
+                  <param name="initial_value">${initial_positions['left_finger_joint']}</param>
+                </state_interface>
             </joint>
         </ros2_control>
